Commit message: Modify urdf to exchange to mjcf.

File: urdf/anymal.urdf (robot description, URDF)
Before this commit: robot anymal, 78 links, 77 joints
Links:
- link LF_FOOT: geometry collision cylinder length=0.282504 radius=0.0175; collision sphere radius=0.03
- link LF_HAA: geometry visual mesh filename=drive.stl scale=1.0 1.0 1.0
- link LF_HFE: geometry collision cylinder length=0.14 radius=0.05; visual mesh filename=drive.stl scale=1.0 1.0 1.0
- link LF_KFE: geometry collision cylinder length=0.14 radius=0.05; visual mesh filename=drive.stl scale=1.0 1.0 1.0
- link LF_hip_fixed: geometry visual mesh filename=hip_l.stl scale=1.0 1.0 1.0
- link LF_shank_fixed: geometry collision box size=0.114998 0.0675 0.04; collision cylinder length=0.04 radius=0.06
- link LF_thigh_fixed: geometry collision box size=0.075 0.06 0.282627; collision cylinder length=0.08 radius=0.065
- link LH_FOOT: geometry collision cylinder length=0.282504 radius=0.0175; collision sphere radius=0.03
- link LH_HAA: geometry visual mesh filename=drive.stl scale=1.0 1.0 1.0
- link LH_HFE: geometry collision cylinder length=0.14 radius=0.05; visual mesh filename=drive.stl scale=1.0 1.0 1.0
- link LH_KFE: geometry collision cylinder length=0.14 radius=0.05; visual mesh filename=drive.stl scale=1.0 1.0 1.0
- link LH_hip_fixed: geometry visual mesh filename=hip_r.stl scale=1.0 1.0 1.0
- link LH_shank_fixed: geometry collision box size=0.114998 0.0675 0.04; collision cylinder length=0.04 radius=0.06
- link LH_thigh_fixed: geometry collision box size=0.075 0.06 0.282627; collision cylinder length=0.08 radius=0.065
- link RF_FOOT: geometry collision cylinder length=0.282504 radius=0.0175; collision sphere radius=0.03
- link RF_HAA: geometry visual mesh filename=drive.stl scale=1.0 1.0 1.0
- link RF_HFE: geometry collision cylinder length=0.14 radius=0.05; visual mesh filename=drive.stl scale=1.0 1.0 1.0
- link RF_KFE: geometry collision cylinder length=0.14 radius=0.05; visual mesh filename=drive.stl scale=1.0 1.0 1.0
- link RF_hip_fixed: geometry visual mesh filename=hip_r.stl scale=1.0 1.0 1.0
- link RF_shank_fixed: geometry collision box size=0.114998 0.0675 0.04; collision cylinder length=0.04 radius=0.06
- link RF_thigh_fixed: geometry collision box size=0.075 0.06 0.282627; collision cylinder length=0.08 radius=0.065
- link RH_FOOT: geometry collision cylinder length=0.282504 radius=0.0175; collision sphere radius=0.03
- link RH_HAA: geometry visual mesh filename=drive.stl scale=1.0 1.0 1.0
- link RH_HFE: geometry collision cylinder length=0.14 radius=0.05; visual mesh filename=drive.stl scale=1.0 1.0 1.0
- link RH_KFE: geometry collision cylinder length=0.14 radius=0.05; visual mesh filename=drive.stl scale=1.0 1.0 1.0
- link RH_hip_fixed: geometry visual mesh filename=hip_l.stl scale=1.0 1.0 1.0
- link RH_shank_fixed: geometry collision box size=0.114998 0.0675 0.04; collision cylinder length=0.04 radius=0.06
- link RH_thigh_fixed: geometry collision box size=0.075 0.06 0.282627; collision cylinder length=0.08 radius=0.065
- link base: geometry collision box size=0.58 0.14 0.18; collision cylinder length=0.145 radius=0.09
- link battery: geometry visual mesh filename=battery.stl scale=1.0 1.0 1.0
- link bottom_shell: geometry visual mesh filename=bottom_shell.stl scale=1.0 1.0 1.0
- link depth_camera_front_camera: geometry visual mesh filename=depth_camera.stl scale=1.0 1.0 1.0
- link depth_camera_left_camera: geometry visual mesh filename=depth_camera.stl scale=1.0 1.0 1.0
- link depth_camera_rear_camera: geometry visual mesh filename=depth_camera.stl scale=1.0 1.0 1.0
- link depth_camera_right_camera: geometry visual mesh filename=depth_camera.stl scale=1.0 1.0 1.0
- link face_front: geometry collision box size=0.11 0.14 0.18; collision cylinder length=0.11 radius=0.09
- link face_rear: geometry collision box size=0.11 0.14 0.18; collision cylinder length=0.11 radius=0.09
- link handle: geometry visual mesh filename=handle.stl scale=1.0 1.0 1.0
- link hatch: geometry visual mesh filename=hatch.stl scale=1.0 1.0 1.0
- link lidar: geometry visual mesh filename=lidar.stl
- link lidar_cage: geometry collision cylinder length=0.12 radius=0.07; visual mesh filename=lidar_cage.stl scale=1.0 1.0 1.0
- link remote: geometry visual mesh filename=remote.stl scale=1.0 1.0 1.0
- link top_shell: geometry visual mesh filename=top_shell.stl scale=1.0 1.0 1.0
- link wide_angle_camera_front_camera: geometry visual mesh filename=wide_angle_camera.stl scale=1.0 1.0 1.0
- link wide_angle_camera_rear_camera: geometry visual mesh filename=wide_angle_camera.stl scale=1.0 1.0 1.0
